Commit message: Update 12/04/2020

File: findchessbot/urdf/planar_3dof.urdf (robot description, URDF)
Before this commit: robot planar_3dof, 6 links, 5 joints
Links:
- removed link end
- removed link gripper
- added link link_3; collision mesh filename=package://lesson_urdf/meshes/link_3.STL; visual mesh filename=package://lesson_urdf/meshes/link_3.STL
- added link link_4; collision mesh filename=package://lesson_urdf/meshes/link_4.STL; visual mesh filename=package://lesson_urdf/meshes/link_4.STL
- link base_link: geometry collision mesh filename=package://lesson_urdf/meshes/base_link.STL; visual mesh filename=package://lesson_urdf/meshes/base_link.STL
- link link_1: mass 1 -> None; geometry collision mesh filename=package://lesson_urdf/meshes/link_1.STL; visual mesh filename=package://lesson_urdf/meshes/link_1.STL
- link link_2: mass 1 -> None; geometry collision mesh filename=package://lesson_urdf/meshes/link_2.STL; visual mesh filename=package://lesson_urdf/meshes/link_2.STL
Joints:
- removed joint gripper_end
- added joint joint_4: type revolute, parent link_3, child link_4, origin xyz=0.315 0 0 rpy=0 0 0, axis 0 0 1, limit lower=-3.14 upper=3.14 effort=0 velocity=0.5
- joint joint_1: origin xyz=0 0 0.05 rpy=0 0 0 -> xyz=0 0 0 rpy=0 0 0
- joint joint_2: limit lower=-1.57 upper=1.57 effort=0 velocity=0.5 -> lower=0 upper=0.1 effort=0 velocity=0.5; origin xyz=0.5 0.0 0.0 rpy=0.0 0 0.0 -> xyz=0 0 0.125 rpy=0 0 0; type revolute -> prismatic
- joint joint_3: child gripper -> link_3; limit lower=-1.57 upper=1.57 effort=0 velocity=0.5 -> lower=-3.14 upper=3.14 effort=0 velocity=0.5; origin xyz=0.5 0.0 0.0 rpy=0.0 0 0.0 -> xyz=0.370 0 0 rpy=0 0 0
