Commit message: Update 8/5/2021

File: findchessbot/urdf/findchessbot.urdf (robot description, URDF)
Before this commit: robot findchessbot, 6 links, 5 joints
Links:
- added link chess_board_black, mass 2.2955; collision mesh filename=package://findchessbot/chessboard_black.STL; visual mesh filename=package://findchessbot/chessboard_black.STL
Joints:
- added joint joint_chess_black: type fixed, parent chess_board, child chess_board_black

Commit message: Update 9/5/2021

File: findchessbot/urdf/findchessbot.urdf (robot description, URDF)
Before this commit: robot findchessbot, 7 links, 6 joints
Links:
- link chess_board_black: mass 2.2955 -> None

Commit message: Update ROS2 pkg

File: findchessbot/urdf/findchessbot.urdf (robot description, URDF)
Before this commit: robot findchessbot, 7 links, 6 joints
Links:
- link base_link: geometry collision mesh filename=package://findchessbot/meshes/base_link.STL; visual mesh filename=package://findchessbot/meshes/base_link.STL
- link chess_board: geometry collision mesh filename=package://findchessbot/meshes/chessboard.STL; visual mesh filename=package://findchessbot/meshes/chessboard.STL
- link chess_board_black: geometry collision mesh filename=package://findchessbot/meshes/chessboard_black.STL; visual mesh filename=package://findchessbot/meshes/chessboard_black.STL
- link link_1: geometry collision mesh filename=package://findchessbot/meshes/link_1.STL; visual mesh filename=package://findchessbot/meshes/link_1.STL
- link link_2: geometry collision mesh filename=package://findchessbot/meshes/link_2.STL; visual mesh filename=package://findchessbot/meshes/link_2.STL
- link link_3: geometry collision mesh filename=package://findchessbot/meshes/link_3.STL; visual mesh filename=package://findchessbot/meshes/link_3.STL
- link link_4: geometry collision mesh filename=package://findchessbot/meshes/link_4.STL; visual mesh filename=package://findchessbot/meshes/link_4.STL
Joints:
- joint joint_chess: origin xyz=0.42744 -0.00059371 0.099999 rpy=0 0 0 -> xyz=0.44 -0.00059371 0.099999 rpy=0 0 0
